File: _autosave-Maxiclaro1.kicad_pcb (KiCad board)
At the start: 2 copper layers, 130.9 x 104.6 mm, 40 parts, among them J1 Screw_Terminal_01x03, J2 ENTRADA, J3 Screw_Terminal_01x03, J4 Screw_Terminal_01x03, J5 Screw_Terminal_01x03, K1 SRD-05VDC-SL-C, K2 SRD-05VDC-SL-C, K3 SRD-05VDC-SL-C, K4 SRD-05VDC-SL-C, Q1 BC547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

Commit message: Add files via upload
Other:
- board size 130.9 x 104.6 mm -> 130.9 x 98.3 mm
Changed lines of the file:
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@@
 	)
 	(gr_rect
-		(start 16.025 29)
+		(start 16.025 35.23)
 		(end 146.92 133.57)
 		(stroke
@@
 		(polygon
 			(pts
-				(xy 16.017183 29) (xy 147.29 29) (xy 147.29 133.749575) (xy 16.06 133.51)
+				(xy 16.019824 35.444508) (xy 146.980318 35.524519) (xy 147.29 133.749575) (xy 16.06 133.51)
 			)
 		)
