File: Maxiclaro1.kicad_pcb (KiCad board)
At the start: 2 copper layers, 130.9 x 104.6 mm, 40 parts, among them J1 Screw_Terminal_01x03, J2 ENTRADA, J3 Screw_Terminal_01x03, J4 Screw_Terminal_01x03, J5 Screw_Terminal_01x03, K1 SRD-05VDC-SL-C, K2 SRD-05VDC-SL-C, K3 SRD-05VDC-SL-C, K4 SRD-05VDC-SL-C, Q1 BC547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

Commit message: Add files via upload
Parts:
- SW1: footprint RB141C1100:SW_RB141C1100 -> 2MS1T1B1M2QES:SW_2MS1T1B1M2QES-5
- U2: footprint Package_TO_SOT_SMD:TO-263-3_TabPin2 -> Package_TO_SOT_SMD:TO-263-2
- moved SW1 5.64 mm to (119.8, 99.5), turned to 180 degrees
Routing:
- net +5V: track 273.5 -> 258.0 mm
- net Net-(J2-Pin_2): track 28.3 -> 16.2 mm
- net Net-(SW1A-B): track 15.1 -> 20.3 mm
Other:
- board size 130.9 x 104.6 mm -> 130.9 x 98.3 mm
Changed lines of the file:
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@@
 		(embedded_fonts no)
 	)
-	(footprint "Package_TO_SOT_SMD:TO-263-3_TabPin2"
+	(footprint "Package_TO_SOT_SMD:TO-263-2"
 		(layer "B.Cu")
 		(at 137.875 83.925)
@@
 		)
 		(fp_line
-			(start -9.325 -0.5)
-			(end -4.625 -0.5)
-			(stroke
-				(width 0.1)
-				(type solid)
-			)
-			(layer "B.Fab")
-		)
-		(fp_line
-			(start -9.325 0.5)
-			(end -9.325 -0.5)
-			(stroke
-				(width 0.1)
-				(type solid)
-			)
-			(layer "B.Fab")
-		)
-		(fp_line
 			(start -9.325 2.04)
 			(end -4.625 2.04)
@@
 		)
 		(fp_line
-			(start -4.625 0.5)
-			(end -9.325 0.5)
-			(stroke
-				(width 0.1)
-				(type solid)
-			)
-			(layer "B.Fab")
-		)
-		(fp_line
 			(start -4.625 3.04)
 			(end -9.325 3.04)
@@
 		)
 		(pad "2" smd roundrect
-			(at -7.65 0)
-			(size 4.6 1.1)
-			(layers "B.Cu" "B.Mask" "B.Paste")
-			(roundrect_rratio 0.227273)
-			(net 9 "GND")
-			(pinfunction "GND")
-			(pintype "power_in")
-		)
-		(pad "2" smd roundrect
 			(at 1.5 0)
 			(size 9.4 10.8)
@@
 		)
 		(embedded_fonts no)
-		(model "${KICAD9_3DMODEL_DIR}/Package_TO_SOT_SMD.3dshapes/TO-263-3_TabPin2.wrl"
+		(model "${KICAD9_3DMODEL_DIR}/Package_TO_SOT_SMD.3dshapes/TO-263-2.wrl"
 			(offset
 				(xyz 0 0 0)
@@
 		)
 	)
-	(footprint "RB141C1100:SW_RB141C1100"
+	(footprint "2MS1T1B1M2QES:SW_2MS1T1B1M2QES-5"
 		(layer "B.Cu")
-		(at 125.43 99.57)
+		(at 119.795 99.53 180)
 		(property "Reference" "SW1"
-			(at -12.575 8.135 0)
+			(at -0.9525 3.4925 0)
 			(layer "B.SilkS")
 			(effects
@@
 		)
 		(property "Value" "SW_DPST_x2"
-			(at -7.495 -8.135 0)
+			(at 7.3025 -3.4925 0)
 			(layer "B.Fab")
 			(effects
@@
 		(attr through_hole)
 		(fp_line
-			(start -16 -7)
-			(end 16 -7)
+			(start 4.065 2.54)
+			(end -4.065 2.54)
 			(stroke
 				(width 0.127)
@@
 		)
 		(fp_line
-			(start -16 7)
-			(end -16 -7)
+			(start 4.065 -2.54)
+			(end 4.065 2.54)
 			(stroke
 				(width 0.127)
@@
 		)
 		(fp_line
-			(start 16 -7)
-			(end 16 7)
+			(start -4.065 2.54)
+			(end -4.065 -2.54)
 			(stroke
 				(width 0.127)
@@
 		)
 		(fp_line
-			(start 16 7)
-			(end -16 7)
+			(start -4.065 -2.54)
+			(end 4.065 -2.54)
 			(stroke
 				(width 0.127)
@@
 		)
 		(fp_circle
-			(center 16.5 0)
-			(end 16.6 0)
+			(center -4.75 0)
+			(end -4.65 0)
 			(stroke
 				(width 0.2)
@@
 		)
 		(fp_line
-			(start -16.25 -7.25)
-			(end 16.25 -7.25)
+			(start 4.315 2.79)
+			(end -4.315 2.79)
 			(stroke
 				(width 0.05)
@@
 		)
 		(fp_line
-			(start -16.25 7.25)
-			(end -16.25 -7.25)
+			(start 4.315 -2.79)
+			(end 4.315 2.79)
 			(stroke
 				(width 0.05)
@@
 		)
 		(fp_line
-			(start 16.25 -7.25)
-			(end 16.25 7.25)
+			(start -4.315 2.79)
+			(end -4.315 -2.79)
 			(stroke
 				(width 0.05)
@@
 		)
 		(fp_line
-			(start 16.25 7.25)
-			(end -16.25 7.25)
+			(start -4.315 -2.79)
+			(end 4.315 -2.79)
 			(stroke
 				(width 0.05)
@@
 		)
 		(fp_line
-			(start -16 -7)
-			(end 16 -7)
+			(start 4.065 2.54)
+			(end -4.065 2.54)
 			(stroke
 				(width 0.127)
@@
 		)
 		(fp_line
-			(start -16 7)
-			(end -16 -7)
+			(start 4.065 -2.54)
+			(end 4.065 2.54)
 			(stroke
 				(width 0.127)
@@
 		)
 		(fp_line
-			(start 16 -7)
-			(end 16 7)
+			(start -4.065 2.54)
+			(end -4.065 -2.54)
 			(stroke
 				(width 0.127)
@@
 		)
 		(fp_line
-			(start 16 7)
-			(end -16 7)
+			(start -4.065 -2.54)
+			(end 4.065 -2.54)
 			(stroke
 				(width 0.127)
@@
 		)
 		(fp_circle
-			(center 16.5 0)
-			(end 16.6 0)
+			(center -4.75 0)
+			(end -4.65 0)
 			(stroke
 				(width 0.2)
@@
 			(layer "B.Fab")
 		)
-		(pad "1" thru_hole oval
-			(at 10.5 0)
-			(size 4.2 8.4)
-			(drill oval 1.2 6.8)
+		(pad "1" thru_hole rect
+			(at -2.54 0 180)
+			(size 1.635 1.635)
+			(drill 1.09)
 			(layers "*.Cu" "*.Mask")
 			(remove_unused_layers no)
@@
 			(solder_mask_margin 0.102)
 		)
-		(pad "2" thru_hole oval
-			(at 0 0)
-			(size 4.2 8.4)
-			(drill oval 1.2 6.8)
+		(pad "2" thru_hole circle
+			(at 0 0 180)
+			(size 1.635 1.635)
+			(drill 1.09)
 			(layers "*.Cu" "*.Mask")
 			(remove_unused_layers no)
@@
 			(solder_mask_margin 0.102)
 		)
+		(pad "3" thru_hole circle
+			(at 2.54 0 180)
+			(size 1.635 1.635)
+			(drill 1.09)
+			(layers "*.Cu" "*.Mask")
+			(remove_unused_layers no)
+			(solder_mask_margin 0.102)
+		)
 		(embedded_fonts no)
 	)
@@
 	)
 	(gr_rect
-		(start 16.025 29)
+		(start 16.025 35.23)
 		(end 146.92 133.57)
 		(stroke
@@
 	)
 	(segment
+		(start 130.225 81.385)
+		(end 124.065 81.385)
+		(width 1)
+		(layer "B.Cu")
+		(net 1)
+	)
+	(segment
 		(start 43.9575 85.12)
 		(end 44.03 85.1925)
@@
 	(segment
 		(start 107.2 84.2)
-		(end 107.2 92.6)
+		(end 107.2 87.65)
 		(width 1)
 		(layer "B.Cu")
@@
 	)
 	(segment
-		(start 130.225 81.385)
-		(end 124.7 81.385)
-		(width 1)
-		(layer "B.Cu")
-		(net 1)
-	)
-	(segment
 		(start 102.6 97.2)
 		(end 102.6 100.81875)
@@
 	)
 	(segment
-		(start 121.45 93.85)
-		(end 121.45 84.635)
+		(start 65.3175 85.1425)
+		(end 66.87 85.1425)
 		(width 1)
 		(layer "B.Cu")
@@
 	)
 	(segment
-		(start 65.3175 85.1425)
-		(end 66.87 85.1425)
+		(start 95.11 85.12)
+		(end 95.11 82.69)
 		(width 1)
 		(layer "B.Cu")
@@
 	)
 	(segment
-		(start 95.11 85.12)
-		(end 95.11 82.69)
+		(start 124.065 81.385)
+		(end 117.8 87.65)
 		(width 1)
 		(layer "B.Cu")
@@
 	)
 	(segment
+		(start 117.8 87.65)
+		(end 107.2 87.65)
+		(width 1)
+		(layer "B.Cu")
+		(net 1)
+	)
+	(segment
 		(start 87.89 85.1325)
 		(end 90.59 85.1325)
@@
 	)
 	(segment
-		(start 61.25 89.21)
-		(end 65.3175 85.1425)
+		(start 107.2 87.65)
+		(end 107.2 92.6)
 		(width 1)
 		(layer "B.Cu")
@@
 	)
 	(segment
-		(start 102.6 100.81875)
-		(end 114.48125 100.81875)
+		(start 61.25 89.21)
+		(end 65.3175 85.1425)
 		(width 1)
 		(layer "B.Cu")
@@
 	)
 	(segment
-		(start 114.48125 100.81875)
-		(end 121.45 93.85)
-		(width 1)
-		(layer "B.Cu")
-		(net 1)
-	)
-	(segment
 		(start 95.05 85.18)
 		(end 95.05 87.11)
@@
 	)
 	(segment
-		(start 121.45 84.635)
-		(end 124.7 81.385)
-		(width 1)
-		(layer "B.Cu")
-		(net 1)
-	)
-	(segment
 		(start 90.6025 85.12)
 		(end 90.59 85.1325)
@@
 	)
 	(segment
-		(start 130.225 89.35)
+		(start 125.285 86.465)
 		(end 130.225 86.465)
 		(width 1)
@@
 	)
 	(segment
-		(start 125.43 94.145)
-		(end 130.225 89.35)
+		(start 119.795 91.955)
+		(end 125.285 86.465)
 		(width 1)
 		(layer "B.Cu")
@@
 	)
 	(segment
-		(start 125.43 99.57)
-		(end 125.43 94.145)
+		(start 119.795 99.53)
+		(end 119.795 91.955)
 		(width 1)
 		(layer "B.Cu")
@@
 	)
 	(segment
-		(start 122.335 115.7)
-		(end 133.5 115.7)
-		(width 1)
-		(layer "B.Cu")
-		(net 46)
-	)
-	(segment
-		(start 135.93 113.27)
-		(end 135.93 99.57)
-		(width 1)
-		(layer "B.Cu")
-		(net 46)
-	)
-	(segment
-		(start 133.5 115.7)
-		(end 135.93 113.27)
+		(start 122.335 99.53)
+		(end 122.335 115.7)
 		(width 1)
 		(layer "B.Cu")
@@
 		(polygon
 			(pts
-				(xy 16.017183 29) (xy 147.29 29) (xy 147.29 133.749575) (xy 16.06 133.51)
+				(xy 16.3 35.5) (xy 146.446432 35.400103) (xy 146.75 133.35) (xy 16.25 133.35)
 			)
 		)
