File: Maxiclaro1/Maxiclaro1.kicad_pcb (KiCad board)
At the start: 2 copper layers, 11 parts, among them K1 SRD-05VDC-SL-C, Q1 BC547

Commit message: Add files via upload
Parts:
- added D3: LED, LED_SMD:LED_0805_2012Metric, B.Cu at (57.1, 79.0)
- added D5: LED, LED_SMD:LED_0805_2012Metric, B.Cu at (38.7, 79.0)
- added D7: LED, LED_SMD:LED_0805_2012Metric, B.Cu at (19.1, 79.0)
- added J1: Screw_Terminal_01x03, TerminalBlock:TerminalBlock_bornier-3_P5.08mm, F.Cu at (73.3, 117.2)
- added J2: ENTRADA, TerminalBlock:TerminalBlock_Altech_AK300-2_P5.00mm, F.Cu at (82.6, 44.8)
- added J3: Screw_Terminal_01x03, TerminalBlock:TerminalBlock_bornier-3_P5.08mm, F.Cu at (55.7, 117.1)
- added J4: Screw_Terminal_01x03, TerminalBlock:TerminalBlock_bornier-3_P5.08mm, F.Cu at (37.8, 117.2)
- added J5: Screw_Terminal_01x03, TerminalBlock:TerminalBlock_bornier-3_P5.08mm, F.Cu at (20.1, 117.2)
- added K2: SRD-05VDC-SL-C, SRD-05VDC-SL-C:RELAY_SRD-05VDC-SL-C, F.Cu at (60.7, 100.0)
- added K3: SRD-05VDC-SL-C, RELAY:RELAY_SRD-05VDC-SL-C, F.Cu at (42.8, 100.2)
- added K4: SRD-05VDC-SL-C, RELAY_SRD-05VDC-SL-C:RELAY_SRD-05VDC-SL-C, F.Cu at (25.1, 100.2)
- added OK2: PC814, PC814:DIL04, B.Cu at (63.2, 74.3)
- added OK3: PC814, DIL04:DIL04, B.Cu at (44.7, 74.3)
- added OK4: PC814, DIL04:DIL04, B.Cu at (25.9, 74.3)
- added Q2: BC547, BC547:SOT95P230X110-3N, B.Cu at (60.7, 87.5)
- added Q3: BC547, BC547:SOT95P230X110-3N, B.Cu at (42.7, 87.4)
- added Q4: BC547, BC547:SOT95P230X110-3N, B.Cu at (25.8, 87.1)
- added R10: 220R, Resistor_SMD:R_0805_2012Metric, B.Cu at (21.3, 69.5)
- added R11: 1K, Resistor_SMD:R_0805_2012Metric, B.Cu at (29.8, 86.2)
- added R12: 220R, Resistor_SMD:R_0805_2012Metric, B.Cu at (19.1, 86.9)
- added R4: 220R, Resistor_SMD:R_0805_2012Metric, B.Cu at (57.9, 69.5)
- added R5: 1K, Resistor_SMD:R_0805_2012Metric, B.Cu at (65.2, 85.6)
- added R6: 220R, Resistor_SMD:R_0805_2012Metric, B.Cu at (57.1, 85.5)
- added R7: 220R, Resistor_SMD:R_0805_2012Metric, B.Cu at (40.1, 69.5)
- added R8: 1K, Resistor_SMD:R_0805_2012Metric, B.Cu at (48.6, 85.7)
- added R9: 220R, Resistor_SMD:R_0805_2012Metric, B.Cu at (38.7, 86.4)
- added SW1: SW_DPST_x2, 2MS1T1B1M2QES:SW_2MS1T1B1M2QES-5, B.Cu at (78.9, 52.6)
- added U1: ESP32-DEVKITC-32D, ESP32−DEVKITC32D:MODULE_ESP32-DEVKITC-32D, F.Cu at (44.5, 50.6)
- added U2: L7805, Package_TO_SOT_SMD:TO-263-2, B.Cu at (59.9, 50.9)
- D1: footprint EESTN5:Led_0805 -> LED_SMD:LED_0805_2012Metric; moved to B.Cu
- D2, D4, D6, D8: footprint OptoDevice:R_LDR_4.9x4.2mm_P2.54mm_Vertical -> Diode_SMD:D_0805_2012Metric; moved to B.Cu
- K1: footprint SRD-05VDC-SL:RELAY_SRD-05VDC-SL-C -> SRD-05VDC-SL-C:RELAY_SRD-05VDC-SL-C
- OK1, Q1: moved to B.Cu
- R1, R2, R3: footprint EESTN5:R_0805 -> Resistor_SMD:R_0805_2012Metric; moved to B.Cu
- moved D8 68.5 mm to (24.6, 82.2), turned to -90 degrees
- moved K1 59.1 mm to (78.3, 99.9), turned to -90 degrees
- moved R2 55.6 mm to (73.5, 69.5), turned to -90 degrees
- moved Q1 55.5 mm to (78.3, 87.3), turned to -90 degrees
- moved D2 51.7 mm to (77.2, 82.6), turned to -90 degrees
- moved OK1 50.4 mm to (78.1, 74.3)
- moved D6 49.8 mm to (43.5, 82.5), turned to -90 degrees
- moved R1 49.1 mm to (82.9, 85.6), turned to -90 degrees
- moved R3 46.3 mm to (72.4, 85.2), turned to 90 degrees
- moved D1 42.8 mm to (72.3, 79.0), turned to 90 degrees
- moved D4 32.6 mm to (61.9, 82.3), turned to -90 degrees
Connections:
- D2 pad 1: Net-(D2-K) -> +5V
- D2 pad 2: +5V -> Net-(D2-A)
- D4 pad 1: Net-(D4-K) -> +5V
- D4 pad 2: +5V -> Net-(D4-A)
- D6 pad 1: Net-(D6-K) -> +5V
- D6 pad 2: +5V -> Net-(D6-A)
- D8 pad 1: Net-(D8-K) -> +5V
- D8 pad 2: +5V -> Net-(D8-A)
- K1 pad A2: Net-(D2-K) -> Net-(D2-A)
- Q1 pad 1: Net-(D2-K) -> Net-(D2-A)
- R3 pad 1: Net-(D2-K) -> Net-(D2-A)
Routing:
- net +5V: track 32.7 -> 220.2 mm
- net INPUT3: track 0.00 -> 33.2 mm
- net GND: track 11.6 -> 39.2 mm
- net COM2: track 0.00 -> 25.8 mm
- net COM: track 0.00 -> 25.4 mm
- net COM1: track 0.00 -> 25.2 mm
- net COM3: track 0.00 -> 25.1 mm
- net Net-(D2-K): track 22.9 -> 0.00 mm
- net INPUT1: track 0.00 -> 19.1 mm
- net Net-(D4-A): track 0.00 -> 16.3 mm
- net Net-(D8-A): track 0.00 -> 16.0 mm
- net Net-(D2-A): track 0.00 -> 15.7 mm
- net Net-(D6-A): track 0.00 -> 15.5 mm
- net Net-(SW1A-B): track 0.00 -> 13.2 mm
- net Net-(J2-Pin_2): track 0.00 -> 13.1 mm
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- added copper zone on B.Cu, net GND
Other:
- board outline added: 77.1 x 89.1 mm
